File: KiCad PCB Design/LCD Board/LCD Board Project/LCD Board Project.kicad_sch (KiCad schematic)
At the start: 8 parts, among them J1 Conn_01x03_Male, J2 Conn_01x03_Male, J3 Conn_01x02_Male, U1 ATtiny412-SS

Commit message: v1.4 - Unknown Updates
Not sure what was changed but I want to push updates.
Parts:
- D1: footprint LED_SMD:LED_2010_5025Metric_Pad1.52x2.65mm_HandSolder -> fab:LED_1206
- J1, J2: footprint Connector_PinHeader_1.00mm:PinHeader_1x03_P1.00mm_Vertical_SMD_Pin1Left -> fab:PinHeader_1x03_P2.54mm_Horizontal_SMD
- J3: footprint Connector_PinHeader_1.00mm:PinHeader_1x02_P1.00mm_Vertical_SMD_Pin1Left -> fab:PinHeader_1x02_P2.54mm_Horizontal_SMD
- R1, R2, R3: footprint Resistor_SMD:R_1206_3216Metric_Pad1.30x1.75mm_HandSolder -> fab:R_1206
Changed lines of the file:
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@@
       (effects (font (size 1.27 1.27)) hide)
     )
-    (property "Footprint" "LED_SMD:LED_2010_5025Metric_Pad1.52x2.65mm_HandSolder" (id 2) (at 172.085 92.71 0)
+    (property "Footprint" "fab:LED_1206" (id 2) (at 172.085 92.71 0)
       (effects (font (size 1.27 1.27)) hide)
     )
@@
       (effects (font (size 1.27 1.27)) (justify left) hide)
     )
-    (property "Footprint" "Connector_PinHeader_1.00mm:PinHeader_1x02_P1.00mm_Vertical_SMD_Pin1Left" (id 2) (at 177.165 74.295 0)
+    (property "Footprint" "fab:PinHeader_1x02_P2.54mm_Horizontal_SMD" (id 2) (at 177.165 74.295 0)
       (effects (font (size 1.27 1.27)) hide)
     )
@@
       (effects (font (size 1.27 1.27)) hide)
     )
-    (property "Footprint" "Resistor_SMD:R_1206_3216Metric_Pad1.30x1.75mm_HandSolder" (id 2) (at 177.292 98.425 90)
+    (property "Footprint" "fab:R_1206" (id 2) (at 177.292 98.425 90)
       (effects (font (size 1.27 1.27)) hide)
     )
@@
       (effects (font (size 1.27 1.27)) hide)
     )
-    (property "Footprint" "Resistor_SMD:R_1206_3216Metric_Pad1.30x1.75mm_HandSolder" (id 2) (at 158.75 69.977 90)
+    (property "Footprint" "fab:R_1206" (id 2) (at 158.75 69.977 90)
       (effects (font (size 1.27 1.27)) hide)
     )
@@
       (effects (font (size 1.27 1.27)) hide)
     )
-    (property "Footprint" "Connector_PinHeader_1.00mm:PinHeader_1x03_P1.00mm_Vertical_SMD_Pin1Left" (id 2) (at 152.4 61.595 0)
+    (property "Footprint" "fab:PinHeader_1x03_P2.54mm_Horizontal_SMD" (id 2) (at 152.4 61.595 0)
       (effects (font (size 1.27 1.27)) hide)
     )
@@
       (effects (font (size 1.27 1.27)) hide)
     )
-    (property "Footprint" "Resistor_SMD:R_1206_3216Metric_Pad1.30x1.75mm_HandSolder" (id 2) (at 158.75 72.517 90)
+    (property "Footprint" "fab:R_1206" (id 2) (at 158.75 72.517 90)
       (effects (font (size 1.27 1.27)) hide)
     )
@@
       (effects (font (size 1.27 1.27)) hide)
     )
-    (property "Footprint" "Connector_PinHeader_1.00mm:PinHeader_1x03_P1.00mm_Vertical_SMD_Pin1Left" (id 2) (at 146.05 112.395 0)
+    (property "Footprint" "fab:PinHeader_1x03_P2.54mm_Horizontal_SMD" (id 2) (at 146.05 112.395 0)
       (effects (font (size 1.27 1.27)) hide)
     )
@@
   (symbol_instances
     (path "/0e6b333e-8992-4c6f-aae2-7a8d485febe6"
-      (reference "D1") (unit 1) (value "LED") (footprint "LED_SMD:LED_2010_5025Metric_Pad1.52x2.65mm_HandSolder")
+      (reference "D1") (unit 1) (value "LED") (footprint "fab:LED_1206")
     )
     (path "/abc5db82-47be-4b8a-8f38-4a13ec4a3f39"
-      (reference "J1") (unit 1) (value "Conn_01x03_Male") (footprint "Connector_PinHeader_1.00mm:PinHeader_1x03_P1.00mm_Vertical_SMD_Pin1Left")
+      (reference "J1") (unit 1) (value "Conn_01x03_Male") (footprint "fab:PinHeader_1x03_P2.54mm_Horizontal_SMD")
     )
     (path "/e2ec72e2-238a-4794-be7b-1b25989146db"
-      (reference "J2") (unit 1) (value "Conn_01x03_Male") (footprint "Connector_PinHeader_1.00mm:PinHeader_1x03_P1.00mm_Vertical_SMD_Pin1Left")
+      (reference "J2") (unit 1) (value "Conn_01x03_Male") (footprint "fab:PinHeader_1x03_P2.54mm_Horizontal_SMD")
     )
     (path "/2b032b6f-8dfd-4462-a7b7-65c2c02e7815"
-      (reference "J3") (unit 1) (value "Conn_01x02_Male") (footprint "Connector_PinHeader_1.00mm:PinHeader_1x02_P1.00mm_Vertical_SMD_Pin1Left")
+      (reference "J3") (unit 1) (value "Conn_01x02_Male") (footprint "fab:PinHeader_1x02_P2.54mm_Horizontal_SMD")
     )
     (path "/9261944e-358a-4351-8027-d100801bf505"
-      (reference "R1") (unit 1) (value "R") (footprint "Resistor_SMD:R_1206_3216Metric_Pad1.30x1.75mm_HandSolder")
+      (reference "R1") (unit 1) (value "R") (footprint "fab:R_1206")
     )
     (path "/baa40f50-b423-496b-a0d4-d95dd791c44d"
-      (reference "R2") (unit 1) (value "R") (footprint "Resistor_SMD:R_1206_3216Metric_Pad1.30x1.75mm_HandSolder")
+      (reference "R2") (unit 1) (value "R") (footprint "fab:R_1206")
     )
     (path "/8ab1171d-54a1-4662-bca2-d8755f4053e1"
-      (reference "R3") (unit 1) (value "R") (footprint "Resistor_SMD:R_1206_3216Metric_Pad1.30x1.75mm_HandSolder")
+      (reference "R3") (unit 1) (value "R") (footprint "fab:R_1206")
     )
     (path "/f33ec0db-ef0f-4576-8054-2833161a8f30"
