File: KiCad PCB Design/RFID Board/RFID Board/RFID Board.kicad_pcb (KiCad board)
At the start: 2 copper layers, 0 parts

Commit message: v1.4 - Unknown Updates
Not sure what was changed but I want to push updates.
Parts:
- added C1: C, fab:C_1206, F.Cu at (154.9, 89.5)
- added D2: LED, fab:LED_1206, F.Cu at (151.8, 91.4)
- added J2: Microcontroller_Ground_UPDI_Power, fab:PinHeader_1x03_P2.54mm_Horizontal_SMD, F.Cu at (158.4, 97.1)
- added J3: SDA SCL, fab:PinHeader_UPDI_01x02_P2.54mm_Horizontal_SMD, F.Cu at (151.7, 100.6)
- added J4: RFID_CC, fab:PinHeader_1x05_P2.54mm_Horizontal_SMD, F.Cu at (138.2, 78.0)
- added J5: Ground_Rail, fab:PinHeader_1x04_P2.54mm_Horizontal_SMD, F.Cu at (158.4, 79.4)
- added J6: Power_Rail, fab:PinHeader_UPDI_01x02_P2.54mm_Horizontal_SMD, F.Cu at (158.4, 90.8)
- added R1: R, fab:R_1206, F.Cu at (146.3, 81.8)
- added R2: R, fab:R_1206, F.Cu at (142.9, 100.3)
- added R3: R, fab:R_1206, F.Cu at (151.1, 84.5)
- added U1: Microcontroller_ATtiny1614-SSFR, fab:SOIC-14_3.9x8.7mm_P1.27mm, F.Cu at (143.1, 92.3)
Routing:
- net Net-(C1-Pad2): track 0.00 -> 103.2 mm
- net Net-(D2-Pad2): track 0.00 -> 67.1 mm
- net Net-(D2-Pad1): track 0.00 -> 39.8 mm
- net Net-(J4-Pad5): track 0.00 -> 17.6 mm
- net Net-(J2-Pad2): track 0.00 -> 17.1 mm
- net Net-(J4-Pad1): track 0.00 -> 16.7 mm
- net Net-(J4-Pad4): track 0.00 -> 15.8 mm
- net Net-(J4-Pad2): track 0.00 -> 15.8 mm
- net Net-(J4-Pad3): track 0.00 -> 13.9 mm
- net Net-(R2-Pad1): track 0.00 -> 11.0 mm
- net Net-(J3-Pad1): track 0.00 -> 10.5 mm
- net Net-(U1-Pad14): track 0.00 -> 7.76 mm
- net Net-(J3-Pad2): track 0.00 -> 6.70 mm
- net Net-(R1-Pad2): track 0.00 -> 3.52 mm
Other:
- board outline added: 35.6 x 39.4 mm
