File: KiCad PCB Design/RFID Board/RFID Board/RFID Board.kicad_sch (KiCad schematic)
At the start: 9 parts, among them J2 Microcontroller_Ground_UPDI_P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, J3 SDA SCL, J4 RFID_CC, J5 Ground_Rail, J6 Power_Rail, U1 Microcontroller_ATtiny1614-SS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

Commit message: v1.4 - Unknown Updates
Not sure what was changed but I want to push updates.
Parts:
- added R1, R3: R, fab:R_1206, symbol fab:R
Connections:
- net at C1.1, D2.1 (K), J2.3 (Pin_3)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: now also R3.1; no longer U1.14 (GND)
- new net: R1.1, U1.14 (GND)
- new net: R1.2, R3.2
Changed lines of the file:
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@@
     (date "2022-04-24")
   )
+  (junction (at 116.84 60.96) (diameter 0) (color 0 0 0 0)
+  )
   (junction (at 110.49 47.625) (diameter 0) (color 0 0 0 1)
   )
@@
   (junction (at 124.46 60.96) (diameter 0) (color 255 0 0 1)
   )
-  (junction (at 118.11 49.53) (diameter 0) (color 0 0 0 1)
-  )
-  (junction (at 116.84 60.96) (diameter 0) (color 0 0 0 1)
+  (junction (at 116.84 49.53) (diameter 0) (color 0 0 0 0)
+  )
+  (wire (pts (xy 101.6 60.96) (xy 107.95 60.96))
+    (stroke (width 0) (type default) (color 0 0 0 0))
   )
   (wire (pts (xy 137.16 60.96) (xy 137.16 81.28))
@@
     (stroke (width 0) (type default) (color 179 0 255 1))
   )
-  (wire (pts (xy 118.11 60.96) (xy 116.84 60.96))
-    (stroke (width 0) (type default) (color 0 0 0 1))
-  )
   (wire (pts (xy 139.065 96.52) (xy 127 96.52))
     (stroke (width 0) (type default) (color 255 142 3 1))
@@
     (stroke (width 0) (type default) (color 0 0 0 1))
   )
+  (wire (pts (xy 107.95 56.515) (xy 107.95 60.96))
+    (stroke (width 0) (type default) (color 0 0 0 0))
+  )
   (wire (pts (xy 123.19 49.53) (xy 139.7 49.53))
     (stroke (width 0) (type default) (color 255 0 2 1))
@@
     (stroke (width 0) (type default) (color 0 0 0 1))
   )
-  (wire (pts (xy 113.03 49.53) (xy 118.11 49.53))
-    (stroke (width 0) (type default) (color 0 0 0 1))
-  )
-  (wire (pts (xy 118.11 49.53) (xy 118.11 60.96))
-    (stroke (width 0) (type default) (color 0 0 0 1))
+  (wire (pts (xy 113.03 49.53) (xy 116.84 49.53))
+    (stroke (width 0) (type default) (color 0 0 0 1))
+  )
+  (wire (pts (xy 116.205 60.96) (xy 116.84 60.96))
+    (stroke (width 0) (type default) (color 0 0 0 0))
   )
   (wire (pts (xy 123.19 49.53) (xy 123.19 60.96))
@@
   (wire (pts (xy 99.695 47.625) (xy 105.41 47.625))
     (stroke (width 0) (type default) (color 0 0 0 1))
+  )
+  (wire (pts (xy 116.84 49.53) (xy 116.84 60.96))
+    (stroke (width 0) (type default) (color 0 0 0 0))
+  )
+  (wire (pts (xy 116.205 58.42) (xy 116.205 56.515))
+    (stroke (width 0) (type default) (color 0 0 0 0))
   )
   (wire (pts (xy 105.41 47.625) (xy 107.95 47.625))
@@
     (stroke (width 0) (type default) (color 179 0 255 1))
   )
+  (wire (pts (xy 108.585 58.42) (xy 108.585 60.96))
+    (stroke (width 0) (type default) (color 0 0 0 0))
+  )
+  (wire (pts (xy 116.205 56.515) (xy 107.95 56.515))
+    (stroke (width 0) (type default) (color 0 0 0 0))
+  )
+  (wire (pts (xy 116.84 49.53) (xy 118.11 49.53))
+    (stroke (width 0) (type default) (color 0 0 0 1))
+  )
   (wire (pts (xy 140.97 97.79) (xy 142.24 97.79))
     (stroke (width 0) (type default) (color 12 0 255 1))
@@
   )
   (wire (pts (xy 99.695 88.9) (xy 99.695 47.625))
-    (stroke (width 0) (type default) (color 0 0 0 1))
-  )
-  (wire (pts (xy 116.84 60.96) (xy 101.6 60.96))
     (stroke (width 0) (type default) (color 0 0 0 1))
   )
@@
     )
     (property "Datasheet" "" (id 3) (at 120.65 60.96 0)
+      (effects (font (size 1.27 1.27)) hide)
+    )
+    (pin "1")
+    (pin "2")
+  )
+  (symbol (lib_id "fab:R") (at 112.395 58.42 270) (unit 1)
+    (in_bom yes) (on_board yes)
+    (property "Reference" "R1" (id 0) (at 112.395 58.42 90))
+    (property "Value" "R" (id 1) (at 112.395 58.42 90)
+      (effects (font (size 1.27 1.27)) hide)
+    )
+    (property "Footprint" "fab:R_1206" (id 2) (at 112.395 56.642 90)
+      (effects (font (size 1.27 1.27)) hide)
+    )
+    (property "Datasheet" "~" (id 3) (at 112.395 58.42 0)
       (effects (font (size 1.27 1.27)) hide)
     )
@@
     )
     (property "Datasheet" "~" (id 3) (at 147.32 97.79 0)
+      (effects (font (size 1.27 1.27)) hide)
+    )
+    (pin "1")
+    (pin "2")
+  )
+  (symbol (lib_id "fab:R") (at 112.395 60.96 270) (unit 1)
+    (in_bom yes) (on_board yes)
+    (property "Reference" "R3" (id 0) (at 112.395 60.96 90))
+    (property "Value" "R" (id 1) (at 112.395 60.96 90)
+      (effects (font (size 1.27 1.27)) hide)
+    )
+    (property "Footprint" "fab:R_1206" (id 2) (at 112.395 59.182 90)
+      (effects (font (size 1.27 1.27)) hide)
+    )
+    (property "Datasheet" "~" (id 3) (at 112.395 60.96 0)
       (effects (font (size 1.27 1.27)) hide)
     )
@@
       (reference "J6") (unit 1) (value "Power_Rail") (footprint "fab:PinHeader_UPDI_01x02_P2.54mm_Horizontal_SMD")
     )
+    (path "/a733cd69-9ed4-4e3b-b218-5bb82fc7ea38"
+      (reference "R1") (unit 1) (value "R") (footprint "fab:R_1206")
+    )
     (path "/67f3a702-954d-41b5-960a-56707a66f2e1"
       (reference "R2") (unit 1) (value "R") (footprint "fab:R_1206")
     )
+    (path "/e1ed2704-639a-4891-a608-30a3fee870f4"
+      (reference "R3") (unit 1) (value "R") (footprint "fab:R_1206")
+    )
     (path "/ed3f6be5-635f-429a-9f31-51d50c3882f0"

Commit message: v1.5 - Code Refactoring & Organization
Other:
- note added: "0 Ohm (Both)"
Changed lines of the file:
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@@
     (stroke (width 0) (type default) (color 0 0 0 1))
+  )
+  (text "0 Ohm (Both)\n" (at 106.045 64.77 0)
+    (effects (font (size 1.27 1.27)) (justify left bottom))
   )
   (symbol (lib_id "fab:Conn_PinHeader_1x02_P2.54mm_Horizontal_SMD") (at 142.24 41.91 270) (unit 1)
