File: KiCad PCB Design/LCD Board 2/LCD Board 2/LCD Board 2.kicad_sch (KiCad schematic)
At the start: 9 parts, among them J1 Conn_PinHeader_1x02_P2.54mm_H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, J2 Conn_PinHeader_1x04_P2.54mm_H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, J2 Conn_PinHeader_1x05_P2.54mm_H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, J3 Conn_PinHeader_1x02_P2.54mm_H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

Commit message: v1.9 - KiCad LCD Board Updates
Parts:
- removed J1: Conn_PinHeader_1x02_P2.54mm_Horizontal_SMD, fab:PinHeader_UPDI_01x02_P2.54mm_Horizontal_SMD, symbol Fab Library:Conn_PinHeader_1x02_P2.54mm_Horizontal_SMD
- removed J2: Conn_PinHeader_1x05_P2.54mm_Horizontal_SMD, fab:PinHeader_1x05_P2.54mm_Horizontal_SMD, symbol Fab Library:Conn_PinHeader_1x05_P2.54mm_Horizontal_SMD
- added J2: Conn_PinHeader_1x10_P2.54mm_Horizontal_SMD, fab:PinHeader_1x10_P2.54mm_Horizontal_SMD, symbol Fab Library:Conn_PinHeader_1x10_P2.54mm_Horizontal_SMD
- added J4: Conn_PinHeader_1x07_P2.54mm_Horizontal_SMD, fab:PinHeader_1x07_P2.54mm_Horizontal_SMD, symbol Fab Library:Conn_PinHeader_1x07_P2.54mm_Horizontal_SMD
- R1, R2: footprint (none) -> fab:R_1206
- gave numbers to parts that had none: 1
- renumbered J2 to J1
Connections:
- net at J1.1 (Pin_1), J1.2 (Pin_2): now also R1.2, U1.8 (PB1/SDA); no longer R2.2, U1.9 (PB0/SCL)
- net at J1.3 (Pin_3), J1.4 (Pin_4): now also R2.2, U1.9 (PB0/SCL); no longer R1.2, U1.8 (PB1/SDA)
- net at R1.1, R2.1: now also J4.1 (Pin_1), J4.2 (Pin_2), J4.3 (Pin_3), J4.4 (Pin_4), J4.5 (Pin_5), J4.6 (Pin_6), J4.7 (Pin_7)
- net at R3.1, U1.14 (GND): now also J2.1 (Pin_1), J2.10 (Pin_10), J2.2 (Pin_2), J2.3 (Pin_3), J2.4 (Pin_4), J2.5 (Pin_5), J2.6 (Pin_6), J2.7 (Pin_7), J2.8 (Pin_8), J2.9 (Pin_9)
Other:
- note added: "4.9k Ohm"
- note added: "Independent - External VCC, Screen VCC, SCL/SDA, and additional VCCs for other screen and RFID to pull from"
- note removed: "Independent - External VCC to Screen VCC && To SCL/SDA"
