File: KiCad PCB Design/Main Board/Main Board/Main Board.kicad_pcb (KiCad board)
At the start: 2 copper layers, 19 x 27.9 mm, 7 parts, among them J1 Conn_01x10_Male, J2 Conn_01x10_Male, J3 Conn_01x10_Male, J4 Conn_01x10_Male, U1 ATtiny412-SS

Commit message: v1.3 - Main PCB Board Updated To Fab Library
Parts:
- D1: footprint LED_SMD:LED_2010_5025Metric_Pad1.52x2.65mm_HandSolder -> fab:LED_1206
- J1, J2, J3, J4: footprint Connector_PinHeader_1.00mm:PinHeader_1x10_P1.00mm_Vertical_SMD_Pin1Left -> fab:PinHeader_1x10_P2.54mm_Horizontal_SMD
- R3: footprint Resistor_SMD:R_1206_3216Metric_Pad1.30x1.75mm_HandSolder -> fab:R_1206
- moved J4 38.6 mm to (197.1, 80.0), turned to 0 degrees
- moved J3 20.3 mm to (191.8, 99.3), turned to -90 degrees
- moved D1 18.8 mm to (184.2, 94.0), turned to 180 degrees
- moved J1 18.4 mm to (162.3, 102.9)
- moved R3 17.9 mm to (184.2, 88.9), turned to 180 degrees
- moved U1 11.3 mm to (176.5, 91.4)
- moved J2 4.79 mm to (168.9, 83.6), turned to 90 degrees
Routing:
- net Net-(J1-Pad1): track 8.03 -> 59.7 mm
- net Net-(J4-Pad1): track 21.0 -> 68.5 mm
- net Net-(J1-Pad10): track 20.0 -> 32.3 mm
- net Net-(J2-Pad1): track 23.7 -> 31.8 mm
- net Net-(J3-Pad1): track 21.1 -> 28.9 mm
- net Net-(D1-Pad1): track 3.49 -> 5.08 mm
- net Net-(D1-Pad2): track 6.36 -> 5.63 mm
Other:
- board size 19 x 27.9 mm -> 52.1 x 33 mm

Commit message: v1.6 - KiCad & Code Additions
Parts:
- added C1: C, fab:C_1206, F.Cu at (174.0, 85.1)
- moved J2 3.81 mm to (168.9, 79.8)
Routing:
- net Net-(J2-Pad1): track 31.8 -> 40.0 mm
- net Net-(J1-Pad1): track 59.7 -> 64.1 mm
- net Net-(J1-Pad10): track 32.3 -> 34.8 mm
Other:
- board size 52.1 x 33 mm -> 52.1 x 36.8 mm
Changed lines of the file:
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@@
     (pad_to_mask_clearance 0)
     (pcbplotparams
-      (layerselection 0x00010fc_ffffffff)
+      (layerselection 0x0001000_7fffffff)
       (disableapertmacros false)
       (usegerberextensions false)
@@
   (net 9 "Net-(J4-Pad1)")
   (footprint "fab:PinHeader_1x10_P2.54mm_Horizontal_SMD" (layer "F.Cu")
-    (at 168.89 83.58 90)
+    (at 168.89 79.77 90)
     (descr "https://s3.amazonaws.com/catalogspreads-pdf/PAGE112-113%20.100%20MALE%20HDR.pdf")
     (tags "horizontal pin header SMD 2.54mm")
@@
     )
   )
+  (footprint "fab:C_1206" (layer "F.Cu")
+    (at 173.99 85.09 90)
+    (descr "Capacitor SMD 1206, hand soldering")
+    (tags "capacitor 1206")
+    (property "Sheetfile" "Main Board.kicad_sch")
+    (property "Sheetname" "")
+    (attr smd)
+    (fp_text reference "C1" (at 0 -1.85 90) (layer "F.SilkS")
+      (effects (font (size 1 1) (thickness 0.15)))
+    )
+    (fp_text value "C" (at 0 1.9 90) (layer "F.Fab")
+      (effects (font (size 1 1) (thickness 0.15)))
+    )
+    (fp_text user "${REFERENCE}" (at 0 0 90) (layer "F.Fab")
+      (effects (font (size 0.7 0.7) (thickness 0.105)))
+    )
+    (fp_line (start 1 1.07) (end -1 1.07) (layer "F.SilkS") (width 0.12))
+    (fp_line (start -1 -1.07) (end 1 -1.07) (layer "F.SilkS") (width 0.12))
+    (fp_line (start -3.25 -1.11) (end -3.25 1.1) (layer "F.CrtYd") (width 0.05))
+    (fp_line (start 3.25 1.1) (end 3.25 -1.11) (layer "F.CrtYd") (width 0.05))
+    (fp_line (start -3.25 -1.11) (end 3.25 -1.11) (layer "F.CrtYd") (width 0.05))
+    (fp_line (start 3.25 1.1) (end -3.25 1.1) (layer "F.CrtYd") (width 0.05))
+    (fp_line (start 1.6 -0.8) (end 1.6 0.8) (layer "F.Fab") (width 0.1))
+    (fp_line (start -1.6 0.8) (end -1.6 -0.8) (layer "F.Fab") (width 0.1))
+    (fp_line (start 1.6 0.8) (end -1.6 0.8) (layer "F.Fab") (width 0.1))
+    (fp_line (start -1.6 -0.8) (end 1.6 -0.8) (layer "F.Fab") (width 0.1))
+    (pad "1" smd rect locked (at -2 0 90) (size 2 1.7) (layers "F.Cu" "F.Paste" "F.Mask")
+      (net 6 "Net-(J1-Pad10)") (pintype "passive"))
+    (pad "2" smd rect locked (at 2 0 90) (size 2 1.7) (layers "F.Cu" "F.Paste" "F.Mask")
+      (net 7 "Net-(J2-Pad1)") (pintype "passive"))
+    (model "${FAB}/fab.3dshapes/C_1206.step"
+      (offset (xyz 0 0 0))
+      (scale (xyz 1 1 1))
+      (rotate (xyz 0 0 0))
+    )
+  )
   (footprint "fab:R_1206" (layer "F.Cu")
     (at 184.15 88.9 180)
@@
     )
   )
-  (gr_line (start 205.74 77.47) (end 205.74 105.41) (layer "Edge.Cuts") (width 0.1))
-  (gr_line (start 156.21 74.93) (end 167.64 74.93) (layer "Edge.Cuts") (width 0.1))
+  (gr_line (start 156.21 71.12) (end 153.67 73.66) (layer "Edge.Cuts") (width 0.1))
+  (gr_line (start 205.74 73.66) (end 205.74 105.41) (layer "Edge.Cuts") (width 0.1))
   (gr_line (start 205.74 105.41) (end 203.2 107.95) (layer "Edge.Cuts") (width 0.1))
   (gr_line (start 156.21 107.95) (end 153.67 105.41) (layer "Edge.Cuts") (width 0.1))
-  (gr_line (start 153.67 105.41) (end 153.67 77.47) (layer "Edge.Cuts") (width 0.1))
+  (gr_line (start 153.67 105.41) (end 153.67 73.66) (layer "Edge.Cuts") (width 0.1))
   (gr_line (start 203.2 107.95) (end 156.21 107.95) (layer "Edge.Cuts") (width 0.1))
-  (gr_line (start 153.67 77.47) (end 156.21 74.93) (layer "Edge.Cuts") (width 0.1))
-  (gr_line (start 167.64 74.93) (end 203.2 74.93) (layer "Edge.Cuts") (width 0.1))
-  (gr_line (start 203.2 74.93) (end 205.74 77.47) (layer "Edge.Cuts") (width 0.1))
-  (segment (start 176.53 88.9) (end 176.53 91.44) (width 0.5) (layer "F.Cu") (net 1))
-  (segment (start 160.02 77.47) (end 163.83 77.47) (width 0.5) (layer "F.Cu") (net 1))
-  (segment (start 166.37 87.63) (end 175.26 87.63) (width 0.5) (layer "F.Cu") (net 1))
-  (segment (start 158.75 101.6) (end 158.75 78.74) (width 0.5) (layer "F.Cu") (net 1))
-  (segment (start 165.1 78.74) (end 165.1 86.36) (width 0.5) (layer "F.Cu") (net 1))
-  (segment (start 160.04 102.89) (end 158.75 101.6) (width 0.5) (layer "F.Cu") (net 1))
-  (segment (start 176.53 91.44) (end 177.165 92.075) (width 0.5) (layer "F.Cu") (net 1))
-  (segment (start 163.83 77.47) (end 165.1 78.74) (width 0.5) (layer "F.Cu") (net 1))
-  (segment (start 165.1 86.36) (end 166.37 87.63) (width 0.5) (layer "F.Cu") (net 1))
-  (segment (start 175.26 87.63) (end 176.53 88.9) (width 0.5) (layer "F.Cu") (net 1))
-  (segment (start 177.165 92.075) (end 179.005 92.075) (width 0.5) (layer "F.Cu") (net 1))
-  (segment (start 158.75 78.74) (end 160.02 77.47) (width 0.5) (layer "F.Cu") (net 1))
-  (segment (start 162.32 102.89) (end 160.04 102.89) (width 0.5) (layer "F.Cu") (net 1))
+  (gr_line (start 167.64 71.12) (end 203.2 71.12) (layer "Edge.Cuts") (width 0.1))
+  (gr_line (start 203.2 71.12) (end 205.74 73.66) (layer "Edge.Cuts") (width 0.1))
+  (gr_line (start 167.64 71.12) (end 156.21 71.12) (layer "Edge.Cuts") (width 0.1))
+  (segment (start 163.83 77.47) (end 160.02 77.47) (width 0.5) (layer "F.Cu") (net 1))
+  (segment (start 176.53 91.44) (end 176.53 86.36) (width 0.5) (layer "F.Cu") (net 1))
+  (segment (start 165.1 78.74) (end 163.83 77.47) (width 0.5) (layer "F.Cu") (net 1))
+  (segment (start 175.26 85.09) (end 172.72 85.09) (width 0.5) (layer "F.Cu") (net 1))
+  (segment (start 165.1 86.36) (end 165.1 78.74) (width 0.5) (layer "F.Cu") (net 1))
+  (segment (start 160.04 102.89) (end 162.32 102.89) (width 0.5) (layer "F.Cu") (net 1))
+  (segment (start 160.02 77.47) (end 158.75 78.74) (width 0.5) (layer "F.Cu") (net 1))
+  (segment (start 171.45 87.63) (end 166.37 87.63) (width 0.5) (layer "F.Cu") (net 1))
+  (segment (start 176.53 86.36) (end 175.26 85.09) (width 0.5) (layer "F.Cu") (net 1))
+  (segment (start 158.75 101.6) (end 160.04 102.89) (width 0.5) (layer "F.Cu") (net 1))
+  (segment (start 158.75 78.74) (end 158.75 101.6) (width 0.5) (layer "F.Cu") (net 1))
+  (segment (start 177.165 92.075) (end 176.53 91.44) (width 0.5) (layer "F.Cu") (net 1))
+  (segment (start 166.37 87.63) (end 165.1 86.36) (width 0.5) (layer "F.Cu") (net 1))
+  (segment (start 172.72 85.09) (end 171.45 86.36) (width 0.5) (layer "F.Cu") (net 1))
+  (segment (start 179.005 92.075) (end 177.165 92.075) (width 0.5) (layer "F.Cu") (net 1))
+  (segment (start 171.45 86.36) (end 171.45 87.63) (width 0.5) (layer "F.Cu") (net 1))
   (segment (start 186.15 88.9) (end 186.15 93.98) (width 0.5) (layer "F.Cu") (net 4))
   (segment (start 182.15 91.98) (end 180.975 90.805) (width 0.5) (layer "F.Cu") (net 5))
@@
   (segment (start 162.975 89.535) (end 174.055 89.535) (width 0.5) (layer "F.Cu") (net 6))
   (segment (start 162.32 80.03) (end 162.32 100.35) (width 0.5) (layer "F.Cu") (net 6))
+  (segment (start 173.99 87.09) (end 173.99 89.47) (width 0.5) (layer "F.Cu") (net 6))
   (segment (start 162.32 90.19) (end 162.975 89.535) (width 0.5) (layer "F.Cu") (net 6))
-  (segment (start 168.89 83.58) (end 191.75 83.58) (width 0.5) (layer "F.Cu") (net 7))
-  (segment (start 181.59 83.58) (end 181.59 88.34) (width 0.5) (layer "F.Cu") (net 7))
+  (segment (start 173.99 89.47) (end 174.055 89.535) (width 0.5) (layer "F.Cu") (net 6))
+  (segment (start 173.99 79.79) (end 173.97 79.77) (width 0.5) (layer "F.Cu") (net 7))
   (segment (start 182.15 88.9) (end 179.64 88.9) (width 0.5) (layer "F.Cu") (net 7))
+  (segment (start 168.89 79.77) (end 191.75 79.77) (width 0.5) (layer "F.Cu") (net 7))
+  (segment (start 173.99 83.09) (end 175.8 83.09) (width 0.5) (layer "F.Cu") (net 7))
+  (segment (start 173.99 83.09) (end 173.99 79.79) (width 0.5) (layer "F.Cu") (net 7))
   (segment (start 179.64 88.9) (end 179.005 89.535) (width 0.5) (layer "F.Cu") (net 7))
+  (segment (start 175.8 83.09) (end 179.005 86.295) (width 0.5) (layer "F.Cu") (net 7))
   (segment (start 181.59 88.34) (end 182.15 88.9) (width 0.5) (layer "F.Cu") (net 7))
+  (segment (start 179.005 86.295) (end 179.005 89.535) (width 0.5) (layer "F.Cu") (net 7))
   (segment (start 191.79 99.3) (end 168.93 99.3) (width 0.5) (layer "F.Cu") (net 8))
   (segment (start 179.09 93.43) (end 179.005 93.345) (width 0.5) (layer "F.Cu") (net 8))

Commit message: v2.0 - i2C Testing Boards Designed
Parts:
- removed C1: C, fab:C_1206
Routing:
- net Net-(J1-Pad10): track 34.8 -> 32.4 mm
Changed lines of the file:
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@@
-    )
-  )
-  (footprint "fab:C_1206" (layer "F.Cu")
-    (at 173.99 85.09 90)
-    (descr "Capacitor SMD 1206, hand soldering")
-    (tags "capacitor 1206")
-    (property "Sheetfile" "Main Board.kicad_sch")
-    (property "Sheetname" "")
-    (attr smd)
-    (fp_text reference "C1" (at 0 -1.85 90) (layer "F.SilkS")
-      (effects (font (size 1 1) (thickness 0.15)))
-    )
-    (fp_text value "C" (at 0 1.9 90) (layer "F.Fab")
-      (effects (font (size 1 1) (thickness 0.15)))
-    )
-    (fp_text user "${REFERENCE}" (at 0 0 90) (layer "F.Fab")
-      (effects (font (size 0.7 0.7) (thickness 0.105)))
-    )
-    (fp_line (start 1 1.07) (end -1 1.07) (layer "F.SilkS") (width 0.12))
-    (fp_line (start -1 -1.07) (end 1 -1.07) (layer "F.SilkS") (width 0.12))
-    (fp_line (start -3.25 -1.11) (end -3.25 1.1) (layer "F.CrtYd") (width 0.05))
-    (fp_line (start 3.25 1.1) (end 3.25 -1.11) (layer "F.CrtYd") (width 0.05))
-    (fp_line (start -3.25 -1.11) (end 3.25 -1.11) (layer "F.CrtYd") (width 0.05))
-    (fp_line (start 3.25 1.1) (end -3.25 1.1) (layer "F.CrtYd") (width 0.05))
-    (fp_line (start 1.6 -0.8) (end 1.6 0.8) (layer "F.Fab") (width 0.1))
-    (fp_line (start -1.6 0.8) (end -1.6 -0.8) (layer "F.Fab") (width 0.1))
-    (fp_line (start 1.6 0.8) (end -1.6 0.8) (layer "F.Fab") (width 0.1))
-    (fp_line (start -1.6 -0.8) (end 1.6 -0.8) (layer "F.Fab") (width 0.1))
-    (pad "1" smd rect locked (at -2 0 90) (size 2 1.7) (layers "F.Cu" "F.Paste" "F.Mask")
-      (net 6 "Net-(J1-Pad10)") (pintype "passive"))
-    (pad "2" smd rect locked (at 2 0 90) (size 2 1.7) (layers "F.Cu" "F.Paste" "F.Mask")
-      (net 7 "Net-(J2-Pad1)") (pintype "passive"))
-    (model "${FAB}/fab.3dshapes/C_1206.step"
-      (offset (xyz 0 0 0))
-      (scale (xyz 1 1 1))
-      (rotate (xyz 0 0 0))
     )
   )
@@
   (segment (start 162.975 89.535) (end 174.055 89.535) (width 0.5) (layer "F.Cu") (net 6))
   (segment (start 162.32 80.03) (end 162.32 100.35) (width 0.5) (layer "F.Cu") (net 6))
-  (segment (start 173.99 87.09) (end 173.99 89.47) (width 0.5) (layer "F.Cu") (net 6))
   (segment (start 162.32 90.19) (end 162.975 89.535) (width 0.5) (layer "F.Cu") (net 6))
   (segment (start 173.99 89.47) (end 174.055 89.535) (width 0.5) (layer "F.Cu") (net 6))
