File: KiCad PCB Design/Main Board/Main Board/Main Board.kicad_sch (KiCad schematic)
At the start: 7 parts, among them J1 Conn_01x10_Male, J2 Conn_01x10_Male, J3 Conn_01x10_Male, J4 Conn_01x10_Male, U1 ATtiny412-SS

Commit message: v1.3 - Main PCB Board Updated To Fab Library
Parts:
- D1: footprint LED_SMD:LED_2010_5025Metric_Pad1.52x2.65mm_HandSolder -> fab:LED_1206
- J1, J2, J3, J4: footprint Connector_PinHeader_1.00mm:PinHeader_1x10_P1.00mm_Vertical_SMD_Pin1Left -> fab:PinHeader_1x10_P2.54mm_Horizontal_SMD
- R3: footprint Resistor_SMD:R_1206_3216Metric_Pad1.30x1.75mm_HandSolder -> fab:R_1206
Changed lines of the file:
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@@
       (effects (font (size 1.27 1.27)) hide)
     )
-    (property "Footprint" "LED_SMD:LED_2010_5025Metric_Pad1.52x2.65mm_HandSolder" (id 2) (at 172.085 92.71 0)
+    (property "Footprint" "fab:LED_1206" (id 2) (at 172.085 92.71 0)
       (effects (font (size 1.27 1.27)) hide)
     )
@@
       (effects (font (size 1.27 1.27)) (justify right) hide)
     )
-    (property "Footprint" "Connector_PinHeader_1.00mm:PinHeader_1x10_P1.00mm_Vertical_SMD_Pin1Left" (id 2) (at 175.895 69.85 0)
+    (property "Footprint" "fab:PinHeader_1x10_P2.54mm_Horizontal_SMD" (id 2) (at 175.895 69.85 0)
       (effects (font (size 1.27 1.27)) hide)
     )
@@
       (effects (font (size 1.27 1.27)) (justify right) hide)
     )
-    (property "Footprint" "Connector_PinHeader_1.00mm:PinHeader_1x10_P1.00mm_Vertical_SMD_Pin1Left" (id 2) (at 143.51 61.595 0)
+    (property "Footprint" "fab:PinHeader_1x10_P2.54mm_Horizontal_SMD" (id 2) (at 143.51 61.595 0)
       (effects (font (size 1.27 1.27)) hide)
     )
@@
       (effects (font (size 1.27 1.27)) hide)
     )
-    (property "Footprint" "Resistor_SMD:R_1206_3216Metric_Pad1.30x1.75mm_HandSolder" (id 2) (at 177.292 98.425 90)
+    (property "Footprint" "fab:R_1206" (id 2) (at 177.292 98.425 90)
       (effects (font (size 1.27 1.27)) hide)
     )
@@
       (effects (font (size 1.27 1.27)) (justify right) hide)
     )
-    (property "Footprint" "Connector_PinHeader_1.00mm:PinHeader_1x10_P1.00mm_Vertical_SMD_Pin1Left" (id 2) (at 146.05 122.555 0)
+    (property "Footprint" "fab:PinHeader_1x10_P2.54mm_Horizontal_SMD" (id 2) (at 146.05 122.555 0)
       (effects (font (size 1.27 1.27)) hide)
     )
@@
       (effects (font (size 1.27 1.27)) (justify right) hide)
     )
-    (property "Footprint" "Connector_PinHeader_1.00mm:PinHeader_1x10_P1.00mm_Vertical_SMD_Pin1Left" (id 2) (at 174.625 44.45 0)
+    (property "Footprint" "fab:PinHeader_1x10_P2.54mm_Horizontal_SMD" (id 2) (at 174.625 44.45 0)
       (effects (font (size 1.27 1.27)) hide)
     )
@@
   (symbol_instances
     (path "/0e6b333e-8992-4c6f-aae2-7a8d485febe6"
-      (reference "D1") (unit 1) (value "LED") (footprint "LED_SMD:LED_2010_5025Metric_Pad1.52x2.65mm_HandSolder")
+      (reference "D1") (unit 1) (value "LED") (footprint "fab:LED_1206")
     )
     (path "/4aaa746c-7db2-4c79-9e3e-5966ae0735f3"
-      (reference "J1") (unit 1) (value "Conn_01x10_Male") (footprint "Connector_PinHeader_1.00mm:PinHeader_1x10_P1.00mm_Vertical_SMD_Pin1Left")
+      (reference "J1") (unit 1) (value "Conn_01x10_Male") (footprint "fab:PinHeader_1x10_P2.54mm_Horizontal_SMD")
     )
     (path "/ada35977-508e-4af9-8821-50f08adb72e4"
-      (reference "J2") (unit 1) (value "Conn_01x10_Male") (footprint "Connector_PinHeader_1.00mm:PinHeader_1x10_P1.00mm_Vertical_SMD_Pin1Left")
+      (reference "J2") (unit 1) (value "Conn_01x10_Male") (footprint "fab:PinHeader_1x10_P2.54mm_Horizontal_SMD")
     )
     (path "/f0c34404-6620-4928-a016-4f27a184298f"
-      (reference "J3") (unit 1) (value "Conn_01x10_Male") (footprint "Connector_PinHeader_1.00mm:PinHeader_1x10_P1.00mm_Vertical_SMD_Pin1Left")
+      (reference "J3") (unit 1) (value "Conn_01x10_Male") (footprint "fab:PinHeader_1x10_P2.54mm_Horizontal_SMD")
     )
     (path "/11d2e56c-5b75-4dbf-9572-c8a39ea65bbc"
-      (reference "J4") (unit 1) (value "Conn_01x10_Male") (footprint "Connector_PinHeader_1.00mm:PinHeader_1x10_P1.00mm_Vertical_SMD_Pin1Left")
+      (reference "J4") (unit 1) (value "Conn_01x10_Male") (footprint "fab:PinHeader_1x10_P2.54mm_Horizontal_SMD")
     )
     (path "/8ab1171d-54a1-4662-bca2-d8755f4053e1"
-      (reference "R3") (unit 1) (value "R") (footprint "Resistor_SMD:R_1206_3216Metric_Pad1.30x1.75mm_HandSolder")
+      (reference "R3") (unit 1) (value "R") (footprint "fab:R_1206")
     )
     (path "/f33ec0db-ef0f-4576-8054-2833161a8f30"

Commit message: v1.6 - KiCad & Code Additions
Parts:
- added C1: C, fab:C_1206, symbol Fab Library:C
Connections:
- net at J1.10 (Pin_10), J1.2 (Pin_2), J1.3 (Pin_3)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: now also C1.1
- net at J2.1 (Pin_1), J2.10 (Pin_10), J2.2 (Pin_2)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: now also C1.2
Changed lines of the file:
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@@
   (junction (at 148.59 66.675) (diameter 0) (color 255 0 0 1)
+  )
+  (junction (at 151.13 73.66) (diameter 0) (color 0 0 0 0)
   )
   (junction (at 169.545 49.53) (diameter 0) (color 255 126 0 1)
@@
     (stroke (width 0) (type default) (color 189 20 255 1))
   )
+  (wire (pts (xy 151.13 73.66) (xy 131.445 73.66))
+    (stroke (width 0) (type default) (color 0 0 0 0))
+  )
   (wire (pts (xy 143.51 66.675) (xy 146.05 66.675))
     (stroke (width 0) (type default) (color 253 0 0 1))
@@
     (stroke (width 0) (type default) (color 3 0 170 1))
   )
-  (wire (pts (xy 151.13 66.675) (xy 151.13 77.47))
+  (wire (pts (xy 131.445 95.25) (xy 131.445 109.855))
+    (stroke (width 0) (type default) (color 0 0 0 0))
+  )
+  (wire (pts (xy 151.13 66.675) (xy 151.13 73.66))
     (stroke (width 0) (type default) (color 255 0 0 1))
   )
@@
     (stroke (width 0) (type default) (color 0 0 0 1))
   )
+  (wire (pts (xy 131.445 109.855) (xy 151.13 109.855))
+    (stroke (width 0) (type default) (color 0 0 0 0))
+  )
   (wire (pts (xy 151.13 122.555) (xy 151.13 125.095))
     (stroke (width 0) (type default) (color 0 0 0 1))
@@
     (stroke (width 0) (type default) (color 0 0 0 1))
   )
+  (wire (pts (xy 151.13 73.66) (xy 151.13 77.47))
+    (stroke (width 0) (type default) (color 255 0 0 1))
+  )
   (wire (pts (xy 166.37 90.17) (xy 169.545 90.17))
     (stroke (width 0) (type default) (color 255 126 0 1))
+  )
+  (wire (pts (xy 131.445 73.66) (xy 131.445 87.63))
+    (stroke (width 0) (type default) (color 0 0 0 0))
   )
   (wire (pts (xy 166.37 85.09) (xy 167.64 85.09))
@@
     (pin "8")
   )
+  (symbol (lib_id "Fab Library:C") (at 131.445 91.44 0) (unit 1)
+    (in_bom yes) (on_board yes) (fields_autoplaced)
+    (property "Reference" "C1" (id 0) (at 134.62 90.1699 0)
+      (effects (font (size 1.27 1.27)) (justify left))
+    )
+    (property "Value" "C" (id 1) (at 134.62 92.7099 0)
+      (effects (font (size 1.27 1.27)) (justify left))
+    )
+    (property "Footprint" "fab:C_1206" (id 2) (at 132.4102 95.25 0)
+      (effects (font (size 1.27 1.27)) hide)
+    )
+    (property "Datasheet" "" (id 3) (at 131.445 91.44 0)
+      (effects (font (size 1.27 1.27)) hide)
+    )
+    (pin "1")
+    (pin "2")
+  )
   (sheet_instances
     (path "/" (page "1"))
   )
   (symbol_instances
+    (path "/f6ed04a0-ba11-4b67-938a-2ac59d652fb6"
+      (reference "C1") (unit 1) (value "C") (footprint "fab:C_1206")
+    )
     (path "/0e6b333e-8992-4c6f-aae2-7a8d485febe6"
       (reference "D1") (unit 1) (value "LED") (footprint "fab:LED_1206")

Commit message: v2.0 - i2C Testing Boards Designed
Parts:
- removed C1: C, fab:C_1206, symbol Fab Library:C
Changed lines of the file:
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@@
   (junction (at 148.59 66.675) (diameter 0) (color 255 0 0 1)
-  )
-  (junction (at 151.13 73.66) (diameter 0) (color 0 0 0 0)
   )
   (junction (at 169.545 49.53) (diameter 0) (color 255 126 0 1)
@@
     (stroke (width 0) (type default) (color 189 20 255 1))
   )
-  (wire (pts (xy 151.13 73.66) (xy 131.445 73.66))
-    (stroke (width 0) (type default) (color 0 0 0 0))
-  )
   (wire (pts (xy 143.51 66.675) (xy 146.05 66.675))
     (stroke (width 0) (type default) (color 253 0 0 1))
@@
     (stroke (width 0) (type default) (color 3 0 170 1))
   )
-  (wire (pts (xy 131.445 95.25) (xy 131.445 109.855))
-    (stroke (width 0) (type default) (color 0 0 0 0))
-  )
-  (wire (pts (xy 151.13 66.675) (xy 151.13 73.66))
+  (wire (pts (xy 170.815 80.01) (xy 170.815 87.63))
+    (stroke (width 0) (type default) (color 189 20 255 1))
+  )
+  (wire (pts (xy 170.815 57.15) (xy 170.815 59.69))
+    (stroke (width 0) (type default) (color 189 20 255 1))
+  )
+  (wire (pts (xy 169.545 31.75) (xy 169.545 34.29))
+    (stroke (width 0) (type default) (color 255 126 0 1))
+  )
+  (wire (pts (xy 151.13 107.95) (xy 151.13 109.855))
+    (stroke (width 0) (type default) (color 0 0 0 1))
+  )
+  (wire (pts (xy 148.59 66.675) (xy 151.13 66.675))
+    (stroke (width 0) (type default) (color 253 0 0 1))
+  )
+  (wire (pts (xy 169.545 34.29) (xy 169.545 36.83))
+    (stroke (width 0) (type default) (color 255 126 0 1))
+  )
+  (wire (pts (xy 151.13 117.475) (xy 151.13 120.015))
+    (stroke (width 0) (type default) (color 0 0 0 1))
+  )
+  (wire (pts (xy 151.13 122.555) (xy 151.13 125.095))
+    (stroke (width 0) (type default) (color 0 0 0 1))
+  )
+  (wire (pts (xy 170.815 67.31) (xy 170.815 69.85))
+    (stroke (width 0) (type default) (color 189 20 255 1))
+  )
+  (wire (pts (xy 130.81 66.675) (xy 133.35 66.675))
+    (stroke (width 0) (type default) (color 253 0 0 1))
+  )
+  (wire (pts (xy 169.545 41.91) (xy 169.545 44.45))
+    (stroke (width 0) (type default) (color 255 126 0 1))
+  )
+  (wire (pts (xy 151.13 125.095) (xy 151.13 127.635))
+    (stroke (width 0) (type default) (color 0 0 0 1))
+  )
+  (wire (pts (xy 151.13 130.175) (xy 151.13 132.715))
+    (stroke (width 0) (type default) (color 0 0 0 1))
+  )
+  (wire (pts (xy 151.13 127.635) (xy 151.13 130.175))
+    (stroke (width 0) (type default) (color 0 0 0 1))
+  )
+  (wire (pts (xy 170.815 77.47) (xy 170.815 80.01))
+    (stroke (width 0) (type default) (color 189 20 255 1))
+  )
+  (wire (pts (xy 169.545 52.07) (xy 169.545 54.61))
+    (stroke (width 0) (type default) (color 255 126 0 1))
+  )
+  (wire (pts (xy 151.13 112.395) (xy 151.13 114.935))
+    (stroke (width 0) (type default) (color 0 0 0 1))
+  )
+  (wire (pts (xy 151.13 66.675) (xy 151.13 77.47))
     (stroke (width 0) (type default) (color 255 0 0 1))
   )
-  (wire (pts (xy 170.815 80.01) (xy 170.815 87.63))
-    (stroke (width 0) (type default) (color 189 20 255 1))
-  )
-  (wire (pts (xy 170.815 57.15) (xy 170.815 59.69))
-    (stroke (width 0) (type default) (color 189 20 255 1))
-  )
-  (wire (pts (xy 169.545 31.75) (xy 169.545 34.29))
-    (stroke (width 0) (type default) (color 255 126 0 1))
-  )
-  (wire (pts (xy 151.13 107.95) (xy 151.13 109.855))
-    (stroke (width 0) (type default) (color 0 0 0 1))
-  )
-  (wire (pts (xy 148.59 66.675) (xy 151.13 66.675))
-    (stroke (width 0) (type default) (color 253 0 0 1))
-  )
-  (wire (pts (xy 169.545 34.29) (xy 169.545 36.83))
-    (stroke (width 0) (type default) (color 255 126 0 1))
-  )
-  (wire (pts (xy 151.13 117.475) (xy 151.13 120.015))
-    (stroke (width 0) (type default) (color 0 0 0 1))
-  )
-  (wire (pts (xy 131.445 109.855) (xy 151.13 109.855))
-    (stroke (width 0) (type default) (color 0 0 0 0))
-  )
-  (wire (pts (xy 151.13 122.555) (xy 151.13 125.095))
-    (stroke (width 0) (type default) (color 0 0 0 1))
-  )
-  (wire (pts (xy 170.815 67.31) (xy 170.815 69.85))
-    (stroke (width 0) (type default) (color 189 20 255 1))
-  )
-  (wire (pts (xy 130.81 66.675) (xy 133.35 66.675))
-    (stroke (width 0) (type default) (color 253 0 0 1))
-  )
-  (wire (pts (xy 169.545 41.91) (xy 169.545 44.45))
-    (stroke (width 0) (type default) (color 255 126 0 1))
-  )
-  (wire (pts (xy 151.13 125.095) (xy 151.13 127.635))
-    (stroke (width 0) (type default) (color 0 0 0 1))
-  )
-  (wire (pts (xy 151.13 130.175) (xy 151.13 132.715))
-    (stroke (width 0) (type default) (color 0 0 0 1))
-  )
-  (wire (pts (xy 151.13 127.635) (xy 151.13 130.175))
-    (stroke (width 0) (type default) (color 0 0 0 1))
-  )
-  (wire (pts (xy 170.815 77.47) (xy 170.815 80.01))
-    (stroke (width 0) (type default) (color 189 20 255 1))
-  )
-  (wire (pts (xy 169.545 52.07) (xy 169.545 54.61))
-    (stroke (width 0) (type default) (color 255 126 0 1))
-  )
-  (wire (pts (xy 151.13 112.395) (xy 151.13 114.935))
-    (stroke (width 0) (type default) (color 0 0 0 1))
-  )
-  (wire (pts (xy 151.13 73.66) (xy 151.13 77.47))
-    (stroke (width 0) (type default) (color 255 0 0 1))
-  )
   (wire (pts (xy 166.37 90.17) (xy 169.545 90.17))
     (stroke (width 0) (type default) (color 255 126 0 1))
-  )
-  (wire (pts (xy 131.445 73.66) (xy 131.445 87.63))
-    (stroke (width 0) (type default) (color 0 0 0 0))
   )
   (wire (pts (xy 166.37 85.09) (xy 167.64 85.09))
@@
     (pin "8")
   )
-  (symbol (lib_id "Fab Library:C") (at 131.445 91.44 0) (unit 1)
-    (in_bom yes) (on_board yes) (fields_autoplaced)
-    (property "Reference" "C1" (id 0) (at 134.62 90.1699 0)
-      (effects (font (size 1.27 1.27)) (justify left))
-    )
-    (property "Value" "C" (id 1) (at 134.62 92.7099 0)
-      (effects (font (size 1.27 1.27)) (justify left))
-    )
-    (property "Footprint" "fab:C_1206" (id 2) (at 132.4102 95.25 0)
-      (effects (font (size 1.27 1.27)) hide)
-    )
-    (property "Datasheet" "" (id 3) (at 131.445 91.44 0)
-      (effects (font (size 1.27 1.27)) hide)
-    )
-    (pin "1")
-    (pin "2")
-  )
   (sheet_instances
     (path "/" (page "1"))
   )
   (symbol_instances
-    (path "/f6ed04a0-ba11-4b67-938a-2ac59d652fb6"
-      (reference "C1") (unit 1) (value "C") (footprint "fab:C_1206")
-    )
     (path "/0e6b333e-8992-4c6f-aae2-7a8d485febe6"
       (reference "D1") (unit 1) (value "LED") (footprint "fab:LED_1206")
