File: i2C Testing/Comms/Comms.kicad_pcb (KiCad board)
At the start: 2 copper layers, 151.1 x 36.1 mm, 21 parts, among them J1 Conn_PinHeader_1x03_P2.54mm_H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, J2 Conn_PinHeader_1x03_P2.54mm_H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, J3 Conn_PinHeader_1x03_P2.54mm_H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, J4 Conn_PinHeader_1x06_P2.54mm_H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, U1 Microcontroller_ATtiny1614-SS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, U2 Microcontroller_ATtiny1614-SS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

Commit message: v2.2 - WORKING I2C
Parts:
- moved U1 109.1 mm to (137.2, 66.1)
- moved R1 109.1 mm to (127.5, 63.6)
- moved R2 109.1 mm to (127.5, 68.6)
- moved D1 109.1 mm to (119.9, 63.6)
- moved D2 109.1 mm to (119.9, 68.6)
- moved J1 109.1 mm to (134.6, 55.7)
- moved J2 109.1 mm to (146.3, 63.5)
Other:
- board size 151.1 x 36.1 mm -> 101 x 74.1 mm
- board text added: "UPDI, Ground, VCC"
- board text removed: "Ground, UPDI, VCC"
