File: LCD RX TX COMBO/KiCad Rx Tx Seven Seg Board/Comms.kicad_sch (KiCad schematic)
At the start: 16 parts, among them J1 Conn_PinHeader_1x03_P2.54mm_H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, J2 Conn_PinHeader_1x02_P2.54mm_H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, J3 Conn_PinHeader_1x03_P2.54mm_H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, J4 Conn_PinHeader_1x02_P2.54mm_H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, U1 Microcontroller_ATtiny1614-SS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, U2 Microcontroller_ATtiny1614-SS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

Commit message: v2.7 - Display Codes & Design
Parts:
- removed D1: LED, fab:LED_1206, symbol Fab Library:LED
- removed J1, J3: Conn_PinHeader_1x03_P2.54mm_Horizontal_SMD, fab:PinHeader_1x03_P2.54mm_Horizontal_SMD, symbol Fab Library:Conn_PinHeader_1x03_P2.54mm_Horizontal_SMD
- removed R1, R5, R6: R, fab:R_1206, symbol Fab Library:R
- added J1: Conn_PinHeader_1x04_P2.54mm_Horizontal_SMD, fab:PinHeader_1x04_P2.54mm_Horizontal_SMD, symbol Fab Library:Conn_PinHeader_1x04_P2.54mm_Horizontal_SMD
Connections:
- net at J4.1: now also U1.9 (PB0/SCL)
- net at J4.2: now also U1.8 (PB1/SDA)
- net at R2.2, U1.14 (GND): now also R3.1, R4.2, U2.14 (GND), J1.1 (Pin_1)
- net at U1.1 (VCC): now also D3.2 (A), U2.1 (VCC), J1.4 (Pin_4)
- net at U1.10 (~{RESET}/UPDI/PA0): now also J1.3 (Pin_3)
- net at U2.10 (~{RESET}/UPDI/PA0): now also J1.2 (Pin_2)
Other:
- note added: "VCC | UPDI Comm. | UPDI Dis. | Ground"
- note removed: "UPDI | Ground | VCC"
- moved on the sheet: D2, D3, D4, J2, J4, R2, R3, R4, U1, U2
