File: New Idea/Primary/Primary.kicad_pcb (KiCad board)
At the start: 2 copper layers, 16 parts, among them J1 Conn_PinHeader_1x03_P2.54mm_H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, J2 Conn_PinHeader_1x06_P2.54mm_H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, J3 Conn_PinHeader_1x08_P2.54mm_V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, U1 Microcontroller_ATtiny1614-SS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

Commit message: v2.9 - KiCad Finished
Parts:
- added J4: Conn_PinHeader_1x03_P2.54mm_Horizontal_SMD, fab:PinHeader_1x03_P2.54mm_Horizontal_SMD, F.Cu at (106.7, 121.9)
- moved R2 3.18 mm to (122.6, 109.2)
- moved D2 1.91 mm to (126.4, 109.2)
Connections:
- J1 pad 3: Net-(J1-Pad3) -> Net-(J2-Pad1)
- J2 pad 5: Net-(J1-Pad3) -> Net-(J2-Pad5)
- J2 pad 6: Net-(J1-Pad3) -> Net-(J2-Pad5)
- R1 pad 1: Net-(J1-Pad3) -> Net-(J2-Pad1)
- R2 pad 1: Net-(J1-Pad3) -> Net-(J2-Pad1)
- R3 pad 1: Net-(J1-Pad3) -> Net-(J2-Pad1)
- R4 pad 1: Net-(J1-Pad3) -> Net-(J2-Pad1)
- R5 pad 1: Net-(J1-Pad3) -> Net-(J2-Pad1)
- R6 pad 1: Net-(J1-Pad3) -> Net-(J2-Pad1)
- U1 pad 14: Net-(J1-Pad3) -> Net-(J2-Pad1)
- U1 pad 9: Net-(J2-Pad1) -> Net-(J2-Pad5)
Routing:
- net Net-(J2-Pad1): track 0.00 -> 111.8 mm
- net Net-(J3-Pad7): track 0.00 -> 52.0 mm
- net Net-(J1-Pad1): track 0.00 -> 16.9 mm
- net Net-(D1-Pad2): track 4.51 -> 18.4 mm
- net Net-(J2-Pad5): track 0.00 -> 13.4 mm
- net Net-(J3-Pad1): track 0.00 -> 9.12 mm
- net Net-(J3-Pad5): track 0.00 -> 9.12 mm
- net Net-(J3-Pad3): track 0.00 -> 8.59 mm
- net Net-(J2-Pad3): track 0.00 -> 8.14 mm
- net Net-(J1-Pad3): track 5.87 -> 0.00 mm
- net Net-(D6-Pad2): track 0.00 -> 5.63 mm
- net Net-(D5-Pad2): track 0.00 -> 5.63 mm
- net Net-(D4-Pad2): track 0.00 -> 5.63 mm
- net Net-(D3-Pad2): track 0.00 -> 5.63 mm
- net Net-(D2-Pad2): track 0.00 -> 5.19 mm
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Other:
- board outline added: 81.3 x 48.3 mm
- board text added: "CONTACTS | GROUNDS"
- board text added: "Control Board"
- board text added: "Debug LED"
- board text added: "EX. VCC | DIS. VCCs"
- board text added: "Flight 282"
- board text added: "GROUND | VCC | UPDI"
- board text added: "Power LED"
- board text added: "SCL | SDA | GROUND"

Commit message: v3.0 - New Board Code
Routing:
- net Net-(J1-Pad1): track 16.9 -> 17.5 mm
Changed lines of the file:
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@@
   (segment (start 159.48 107.95) (end 163.1 107.95) (width 0.5) (layer "F.Cu") (net 9))
   (segment (start 149.845 107.95) (end 155.48 107.95) (width 0.5) (layer "F.Cu") (net 10))
-  (segment (start 132.2832 104.3432) (end 133.35 105.41) (width 0.5) (layer "F.Cu") (net 11))
-  (segment (start 133.35 105.41) (end 133.35 109.22) (width 0.5) (layer "F.Cu") (net 11))
+  (segment (start 129.54 103.6828) (end 130.2004 104.3432) (width 0.5) (layer "F.Cu") (net 11))
+  (segment (start 134.62 110.49) (end 135.89 110.49) (width 0.5) (layer "F.Cu") (net 11))
   (segment (start 131.054 98.82) (end 129.54 100.334) (width 0.5) (layer "F.Cu") (net 11))
-  (segment (start 130.2004 104.3432) (end 132.2832 104.3432) (width 0.5) (layer "F.Cu") (net 11))
+  (segment (start 129.54 100.334) (end 129.54 103.6828) (width 0.5) (layer "F.Cu") (net 11))
+  (segment (start 130.2004 104.3432) (end 133.35 104.3432) (width 0.5) (layer "F.Cu") (net 11))
   (segment (start 133.35 109.22) (end 134.62 110.49) (width 0.5) (layer "F.Cu") (net 11))
-  (segment (start 134.62 110.49) (end 135.89 110.49) (width 0.5) (layer "F.Cu") (net 11))
-  (segment (start 129.54 103.6828) (end 130.2004 104.3432) (width 0.5) (layer "F.Cu") (net 11))
-  (segment (start 129.54 100.334) (end 129.54 103.6828) (width 0.5) (layer "F.Cu") (net 11))
+  (segment (start 133.35 104.3432) (end 133.35 109.22) (width 0.5) (layer "F.Cu") (net 11))
   (segment (start 133.35 114.3) (end 133.35 112.395) (width 0.5) (layer "F.Cu") (net 12))
   (segment (start 133.35 112.395) (end 133.985 111.76) (width 0.5) (layer "F.Cu") (net 12))

Commit message: v3.1 - Board Updates
Parts:
- removed D3, D4, D5, D6: LED, fab:LED_1206
- removed R3, R4, R5, R6: R, fab:R_1206
- J1: value Conn_PinHeader_1x03_P2.54mm_Horizontal_SMD -> Conn_PinHeader_1x04_P2.54mm_Horizontal_SMD; footprint fab:PinHeader_1x03_P2.54mm_Horizontal_SMD -> fab:PinHeader_1x04_P2.54mm_Horizontal_SMD
- J4: value Conn_PinHeader_1x03_P2.54mm_Horizontal_SMD -> Conn_PinHeader_1x05_P2.54mm_Horizontal_SMD; footprint fab:PinHeader_1x03_P2.54mm_Horizontal_SMD -> fab:PinHeader_1x05_P2.54mm_Horizontal_SMD
- moved J4 0.24 mm to (106.4, 121.9)
- moved J1 0.23 mm to (130.8, 98.8)
Connections:
- J3 pad 2: Net-(D4-Pad2) -> Net-(J2-Pad1)
- J3 pad 4: Net-(D6-Pad2) -> Net-(J2-Pad1)
- J3 pad 6: Net-(D5-Pad2) -> Net-(J2-Pad1)
- J3 pad 8: Net-(D3-Pad2) -> Net-(J2-Pad1)
Routing:
- net Net-(J2-Pad1): track 111.8 -> 74.2 mm
- net Net-(D6-Pad2): track 5.63 -> 0.00 mm
- net Net-(D5-Pad2): track 5.63 -> 0.00 mm
- net Net-(D4-Pad2): track 5.63 -> 0.00 mm
- net Net-(D3-Pad2): track 5.63 -> 0.00 mm
- net Net-(J4-Pad1): track 5.08 -> 10.2 mm
- net Net-(D6-Pad1): track 3.62 -> 0.00 mm
- net Net-(D5-Pad1): track 3.62 -> 0.00 mm
- net Net-(D4-Pad1): track 3.62 -> 0.00 mm
- net Net-(D3-Pad1): track 3.62 -> 0.00 mm
Other:
- board text added: "GROUNDs | VCC | UPDI"
- board text removed: "GROUND | VCC | UPDI"
