File: New Idea/Primary/Primary.kicad_sch (KiCad schematic)
At the start: 16 parts, among them J1 Conn_PinHeader_1x03_P2.54mm_H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, J2 Conn_PinHeader_1x06_P2.54mm_H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, J3 Conn_PinHeader_1x08_P2.54mm_V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, U1 Microcontroller_ATtiny1614-SS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

Commit message: v2.9 - KiCad Finished
Parts:
- added J4: Conn_PinHeader_1x03_P2.54mm_Horizontal_SMD, fab:PinHeader_1x03_P2.54mm_Horizontal_SMD, symbol Fab Library:Conn_PinHeader_1x03_P2.54mm_Horizontal_SMD
Connections:
- net at J1.3 (Pin_3), R1.1, R2.1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: now also J2.1 (Pin_1), J2.2 (Pin_2); no longer J2.5 (Pin_5), J2.6 (Pin_6)
- new net: J2.5 (Pin_5), J2.6 (Pin_6), U1.9 (PB0/SCL)
- new net: J4.1 (Pin_1), J4.2 (Pin_2), J4.3 (Pin_3)
Other:
- note added: "External VCC to Seven Segment VCCs"
Changed lines of the file:
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@@
   (junction (at 173.355 116.205) (diameter 0) (color 0 0 0 0)
   )
-  (junction (at 134.62 100.965) (diameter 0) (color 0 0 0 0)
-  )
   (junction (at 126.365 89.535) (diameter 0) (color 0 0 0 0)
   )
   (junction (at 173.355 111.125) (diameter 0) (color 0 0 0 0)
   )
-  (junction (at 134.62 98.425) (diameter 0) (color 0 0 0 0)
-  )
-  (junction (at 126.365 112.395) (diameter 0) (color 0 0 0 0)
+  (junction (at 133.35 106.045) (diameter 0) (color 0 0 0 0)
   )
   (junction (at 151.13 129.54) (diameter 0) (color 0 0 0 0)
   )
-  (junction (at 134.62 108.585) (diameter 0) (color 0 0 0 0)
+  (junction (at 126.365 92.71) (diameter 0) (color 0 0 0 0)
+  )
+  (junction (at 133.35 95.885) (diameter 0) (color 0 0 0 0)
   )
   (junction (at 173.355 106.045) (diameter 0) (color 0 0 0 0)
@@
   (junction (at 151.13 86.36) (diameter 0) (color 0 0 0 0)
   )
+  (junction (at 173.355 86.36) (diameter 0) (color 0 0 0 0)
+  )
+  (junction (at 133.35 100.965) (diameter 0) (color 0 0 0 0)
+  )
   (wire (pts (xy 191.135 100.965) (xy 192.405 100.965))
     (stroke (width 0) (type default) (color 0 0 0 0))
@@
     (stroke (width 0) (type default) (color 0 0 0 0))
   )
-  (wire (pts (xy 134.62 95.885) (xy 133.35 95.885))
-    (stroke (width 0) (type default) (color 0 0 0 0))
-  )
   (wire (pts (xy 151.13 78.74) (xy 151.13 86.36))
     (stroke (width 0) (type default) (color 0 0 0 0))
   )
+  (wire (pts (xy 135.89 98.425) (xy 134.62 98.425))
+    (stroke (width 0) (type default) (color 0 0 0 0))
+  )
   (wire (pts (xy 173.355 106.045) (xy 174.625 106.045))
     (stroke (width 0) (type default) (color 0 0 0 0))
@@
     (stroke (width 0) (type default) (color 0 0 0 0))
   )
+  (wire (pts (xy 133.35 100.965) (xy 133.35 103.505))
+    (stroke (width 0) (type default) (color 0 0 0 0))
+  )
   (wire (pts (xy 173.355 106.045) (xy 173.355 111.125))
     (stroke (width 0) (type default) (color 0 0 0 0))
   )
-  (wire (pts (xy 134.62 108.585) (xy 134.62 112.395))
+  (wire (pts (xy 134.62 98.425) (xy 134.62 106.045))
+    (stroke (width 0) (type default) (color 0 0 0 0))
+  )
+  (wire (pts (xy 133.35 98.425) (xy 133.35 95.885))
+    (stroke (width 0) (type default) (color 0 0 0 0))
+  )
+  (wire (pts (xy 133.35 95.885) (xy 133.35 92.71))
+    (stroke (width 0) (type default) (color 0 0 0 0))
+  )
+  (wire (pts (xy 170.815 86.36) (xy 173.355 86.36))
     (stroke (width 0) (type default) (color 0 0 0 0))
   )
@@
     (stroke (width 0) (type default) (color 0 0 0 0))
   )
-  (wire (pts (xy 126.365 89.535) (xy 126.365 112.395))
-    (stroke (width 0) (type default) (color 0 0 0 0))
-  )
-  (wire (pts (xy 134.62 100.965) (xy 135.89 100.965))
+  (wire (pts (xy 133.35 106.045) (xy 133.35 108.585))
+    (stroke (width 0) (type default) (color 0 0 0 0))
+  )
+  (wire (pts (xy 126.365 89.535) (xy 126.365 92.71))
     (stroke (width 0) (type default) (color 0 0 0 0))
   )
@@
     (stroke (width 0) (type default) (color 0 0 0 0))
   )
-  (wire (pts (xy 134.62 103.505) (xy 133.35 103.505))
+  (wire (pts (xy 134.62 106.045) (xy 133.35 106.045))
     (stroke (width 0) (type default) (color 0 0 0 0))
   )
@@
     (stroke (width 0) (type default) (color 0 0 0 0))
   )
-  (wire (pts (xy 126.365 112.395) (xy 126.365 129.54))
-    (stroke (width 0) (type default) (color 0 0 0 0))
-  )
   (wire (pts (xy 166.37 106.045) (xy 171.45 106.045))
     (stroke (width 0) (type default) (color 0 0 0 0))
@@
     (stroke (width 0) (type default) (color 0 0 0 0))
   )
+  (wire (pts (xy 135.89 100.965) (xy 133.35 100.965))
+    (stroke (width 0) (type default) (color 0 0 0 0))
+  )
   (wire (pts (xy 191.135 111.125) (xy 192.405 111.125))
     (stroke (width 0) (type default) (color 0 0 0 0))
@@
     (stroke (width 0) (type default) (color 0 0 0 0))
   )
+  (wire (pts (xy 126.365 92.71) (xy 126.365 129.54))
+    (stroke (width 0) (type default) (color 0 0 0 0))
+  )
   (wire (pts (xy 167.005 98.425) (xy 166.37 98.425))
     (stroke (width 0) (type default) (color 0 0 0 0))
@@
     (stroke (width 0) (type default) (color 0 0 0 0))
   )
-  (wire (pts (xy 134.62 100.965) (xy 133.35 100.965))
-    (stroke (width 0) (type default) (color 0 0 0 0))
-  )
-  (wire (pts (xy 134.62 106.045) (xy 133.35 106.045))
+  (wire (pts (xy 173.355 86.36) (xy 175.895 86.36))
     (stroke (width 0) (type default) (color 0 0 0 0))
   )
@@
     (stroke (width 0) (type default) (color 0 0 0 0))
   )
-  (wire (pts (xy 134.62 112.395) (xy 126.365 112.395))
+  (wire (pts (xy 133.35 92.71) (xy 126.365 92.71))
     (stroke (width 0) (type default) (color 0 0 0 0))
   )
@@
     (stroke (width 0) (type default) (color 0 0 0 0))
   )
-  (wire (pts (xy 134.62 98.425) (xy 133.35 98.425))
-    (stroke (width 0) (type default) (color 0 0 0 0))
-  )
   (wire (pts (xy 172.72 108.585) (xy 192.405 108.585))
     (stroke (width 0) (type default) (color 0 0 0 0))
   )
-  (wire (pts (xy 134.62 98.425) (xy 135.89 98.425))
-    (stroke (width 0) (type default) (color 0 0 0 0))
-  )
-  (wire (pts (xy 134.62 100.965) (xy 134.62 103.505))
-    (stroke (width 0) (type default) (color 0 0 0 0))
-  )
   (wire (pts (xy 153.67 89.535) (xy 167.005 89.535))
     (stroke (width 0) (type default) (color 0 0 0 0))
@@
     (stroke (width 0) (type default) (color 0 0 0 0))
   )
-  (wire (pts (xy 134.62 106.045) (xy 134.62 108.585))
-    (stroke (width 0) (type default) (color 0 0 0 0))
-  )
-  (wire (pts (xy 134.62 95.885) (xy 134.62 98.425))
-    (stroke (width 0) (type default) (color 0 0 0 0))
-  )
   (wire (pts (xy 153.67 78.74) (xy 153.67 89.535))
     (stroke (width 0) (type default) (color 0 0 0 0))
@@
     (stroke (width 0) (type default) (color 0 0 0 0))
   )
-  (wire (pts (xy 134.62 108.585) (xy 133.35 108.585))
-    (stroke (width 0) (type default) (color 0 0 0 0))
-  )
   (text "Power LED" (at 132.715 84.455 0)
+    (effects (font (size 1.27 1.27)) (justify left bottom))
+  )
+  (text "External VCC to Seven Segment VCCs" (at 176.53 84.455 0)
     (effects (font (size 1.27 1.27)) (justify left bottom))
   )
@@
     (pin "9")
   )
+  (symbol (lib_id "Fab Library:Conn_PinHeader_1x03_P2.54mm_Horizontal_SMD") (at 173.355 81.28 270) (unit 1)
+    (in_bom yes) (on_board yes)
+    (property "Reference" "J4" (id 0) (at 173.355 79.375 90))
+    (property "Value" "Conn_PinHeader_1x03_P2.54mm_Horizontal_SMD" (id 1) (at 173.355 78.105 90)
+      (effects (font (size 1.27 1.27)) hide)
+    )
+    (property "Footprint" "fab:PinHeader_1x03_P2.54mm_Horizontal_SMD" (id 2) (at 173.355 81.28 0)
+      (effects (font (size 1.27 1.27)) hide)
+    )
+    (property "Datasheet" "~" (id 3) (at 173.355 81.28 0)
+      (effects (font (size 1.27 1.27)) hide)
+    )
+    (pin "1")
+    (pin "2")
+    (pin "3")
+  )
   (symbol (lib_id "Fab Library:LED") (at 145.415 86.36 0) (unit 1)
     (in_bom yes) (on_board yes)
@@
       (reference "J3") (unit 1) (value "Conn_PinHeader_1x08_P2.54mm_Vertical_THT_D1.4mm") (footprint "fab:PinHeader_2x04_P2.54mm_Vertical_SMD")
     )
+    (path "/b9d13894-fa1c-4284-9d8b-e905ac2bc28e"
+      (reference "J4") (unit 1) (value "Conn_PinHeader_1x03_P2.54mm_Horizontal_SMD") (footprint "fab:PinHeader_1x03_P2.54mm_Horizontal_SMD")
+    )
     (path "/58f03de9-1217-45a3-bd60-63df77c4f469"

Commit message: v3.1 - Board Updates
Parts:
- removed D3, D4, D5, D6: LED, fab:LED_1206, symbol Fab Library:LED
- removed J1, J4: Conn_PinHeader_1x03_P2.54mm_Horizontal_SMD, fab:PinHeader_1x03_P2.54mm_Horizontal_SMD, symbol Fab Library:Conn_PinHeader_1x03_P2.54mm_Horizontal_SMD
- removed R3, R4, R5, R6: R, fab:R_1206, symbol Fab Library:R
- added J1: Conn_PinHeader_1x04_P2.54mm_Horizontal_SMD, fab:PinHeader_1x04_P2.54mm_Horizontal_SMD, symbol Fab Library:Conn_PinHeader_1x04_P2.54mm_Horizontal_SMD
- added J4: Conn_PinHeader_1x05_P2.54mm_Horizontal_SMD, fab:PinHeader_1x05_P2.54mm_Horizontal_SMD, symbol Fab Library:Conn_PinHeader_1x05_P2.54mm_Horizontal_SMD
Connections:
- net at J3.6 (Pin_6): now also J2.1 (Pin_1), J2.2 (Pin_2), J3.2 (Pin_2), J3.4 (Pin_4), J3.8 (Pin_8), R1.1, R2.1, U1.14 (GND), J1.3 (Pin_3), J1.4 (Pin_4)
- net at D1.2 (A), U1.1 (VCC): now also J1.2 (Pin_2)
- net at U1.10 (~{RESET}/UPDI/PA0): now also J1.1 (Pin_1)
- new net: J4.1 (Pin_1), J4.2 (Pin_2), J4.3 (Pin_3), J4.4 (Pin_4), J4.5 (Pin_5)
