File: New Idea/Power/Power/Power.kicad_pcb (KiCad board)
At the start: 2 copper layers, 48.3 x 30.5 mm, 3 parts, among them J1 Conn_PinHeader_1x02_P2.54mm_H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, J2 Conn_PinHeader_1x04_P2.54mm_H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, U1 Regulator_Linear_NCP1117-5.0V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

Commit message: v3.4 - KiCad and Code Updates
Parts:
- moved J2 16.8 mm to (123.2, 101.8), turned to -90 degrees
- moved U1 11.1 mm to (106.7, 94.0)
- moved J1 3.92 mm to (91.4, 101.6)
Routing:
- net Net-(J1-Pad1): track 5.75 -> 14.3 mm
- net Net-(J1-Pad2): track 37.9 -> 43.7 mm
- net Net-(J2-Pad3): track 18.1 -> 19.1 mm
Changed lines of the file:
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@@
   (net 3 "Net-(J2-Pad3)")
   (footprint "fab:SOT-223-3_TabPin2" (layer "F.Cu")
-    (at 96.495 98.425)
+    (at 106.68 93.98)
     (descr "module CMS SOT223 4 pins")
     (tags "CMS SOT")
@@
   )
   (footprint "fab:PinHeader_1x04_P2.54mm_Horizontal_SMD" (layer "F.Cu")
-    (at 108.345 93.98)
+    (at 123.18 101.84 -90)
     (descr "https://s3.amazonaws.com/catalogspreads-pdf/PAGE112-113%20.100%20MALE%20HDR.pdf")
     (tags "horizontal pin header SMD 2.54mm")
@@
     (property "Sheetname" "")
     (attr smd)
-    (fp_text reference "J2" (at -1.524 -2.54) (layer "F.SilkS")
-      (effects (font (size 1 1) (thickness 0.15)) (justify right))
+    (fp_text reference "J2" (at -1.524 -2.54 90) (layer "F.SilkS")
+      (effects (font (size 1 1) (thickness 0.15)) (justify left))
     )
-    (fp_text value "Conn_PinHeader_1x04_P2.54mm_Horizontal_SMD" (at 0 10.795) (layer "F.Fab")
+    (fp_text value "Conn_PinHeader_1x04_P2.54mm_Horizontal_SMD" (at 0 10.795 90) (layer "F.Fab")
       (effects (font (size 1 1) (thickness 0.15)))
     )
-    (fp_text user "${REFERENCE}" (at 2.5 3.9 90) (layer "F.Fab")
+    (fp_text user "${REFERENCE}" (at 2.5 3.9) (layer "F.Fab")
       (effects (font (size 1 1) (thickness 0.15)))
     )
@@
     (fp_line (start 6.34 -1.27) (end 6.35 8.89) (layer "F.Fab") (width 0.1))
     (fp_line (start 3.81 0) (end -0.635 0) (layer "F.Fab") (width 0.1))
-    (pad "1" smd rect locked (at 0 0) (size 2.5 1.7) (layers "F.Cu" "F.Paste" "F.Mask")
+    (pad "1" smd rect locked (at 0 0 270) (size 2.5 1.7) (layers "F.Cu" "F.Paste" "F.Mask")
       (net 2 "Net-(J1-Pad2)") (pinfunction "Pin_1") (pintype "passive"))
-    (pad "2" smd rect locked (at 0 2.54) (size 2.5 1.7) (layers "F.Cu" "F.Paste" "F.Mask")
+    (pad "2" smd rect locked (at 0 2.54 270) (size 2.5 1.7) (layers "F.Cu" "F.Paste" "F.Mask")
       (net 2 "Net-(J1-Pad2)") (pinfunction "Pin_2") (pintype "passive"))
-    (pad "3" smd rect locked (at 0 5.08) (size 2.5 1.7) (layers "F.Cu" "F.Paste" "F.Mask")
+    (pad "3" smd rect locked (at 0 5.08 270) (size 2.5 1.7) (layers "F.Cu" "F.Paste" "F.Mask")
       (net 3 "Net-(J2-Pad3)") (pinfunction "Pin_3") (pintype "passive"))
-    (pad "4" smd rect locked (at 0 7.62) (size 2.5 1.7) (layers "F.Cu" "F.Paste" "F.Mask")
+    (pad "4" smd rect locked (at 0 7.62 270) (size 2.5 1.7) (layers "F.Cu" "F.Paste" "F.Mask")
       (net 3 "Net-(J2-Pad3)") (pinfunction "Pin_4") (pintype "passive"))
     (model "${FAB}/fab.3dshapes/Header_SMD_01x04_P2.54mm_Horizontal_Male.step"
@@
   )
   (footprint "fab:PinHeader_UPDI_01x02_P2.54mm_Horizontal_SMD" (layer "F.Cu")
-    (at 88.025 99.675 180)
+    (at 91.44 101.6 180)
     (descr "https://s3.amazonaws.com/catalogspreads-pdf/PAGE112-113%20.100%20MALE%20HDR.pdf")
     (tags "horizontal pin header SMD 2.54mm")
@@
   (gr_line (start 127 81.28) (end 127 106.68) (layer "Edge.Cuts") (width 0.1))
   (gr_arc (start 78.74 81.28) (mid 79.483949 79.483949) (end 81.28 78.74) (layer "Edge.Cuts") (width 0.1))
-  (gr_text "VCC" (at 88.025 104.14) (layer "F.Cu")
+  (gr_text "VCC" (at 91.44 106.68) (layer "F.Cu")
     (effects (font (size 1.5 1.5) (thickness 0.3)))
   )
@@
     (effects (font (size 3 3) (thickness 0.5)))
   )
-  (gr_text "Ground" (at 120.904 95.885) (layer "F.Cu")
+  (gr_text "Ground" (at 121.92 96.52) (layer "F.Cu")
     (effects (font (size 1.5 1.5) (thickness 0.3)))
   )
-  (gr_text "Ground" (at 87.63 92.71) (layer "F.Cu")
+  (gr_text "Ground" (at 91.44 93.98) (layer "F.Cu")
     (effects (font (size 1.5 1.5) (thickness 0.3)))
   )
-  (gr_text "VCC" (at 119.38 101.092) (layer "F.Cu")
+  (gr_text "VCC" (at 109.22 104.14) (layer "F.Cu")
     (effects (font (size 1.5 1.5) (thickness 0.3)))
   )
-  (segment (start 88.025 99.675) (end 89.515 99.675) (width 0.5) (layer "F.Cu") (net 1))
-  (segment (start 89.515 99.675) (end 90.565 100.725) (width 0.5) (layer "F.Cu") (net 1))
-  (segment (start 90.565 100.725) (end 93.345 100.725) (width 0.5) (layer "F.Cu") (net 1))
-  (segment (start 93.345 93.98) (end 93.98 93.345) (width 0.5) (layer "F.Cu") (net 2))
-  (segment (start 90.565 96.125) (end 93.345 96.125) (width 0.5) (layer "F.Cu") (net 2))
-  (segment (start 93.345 96.125) (end 93.345 93.98) (width 0.5) (layer "F.Cu") (net 2))
-  (segment (start 108.345 97.145) (end 111.75 97.145) (width 0.5) (layer "F.Cu") (net 2))
-  (segment (start 88.025 97.135) (end 89.555 97.135) (width 0.5) (layer "F.Cu") (net 2))
-  (segment (start 89.555 97.135) (end 90.565 96.125) (width 0.5) (layer "F.Cu") (net 2))
-  (segment (start 102.235 91.44) (end 109.855 91.44) (width 0.5) (layer "F.Cu") (net 2))
-  (segment (start 100.33 93.345) (end 102.235 91.44) (width 0.5) (layer "F.Cu") (net 2))
-  (segment (start 93.98 93.345) (end 100.33 93.345) (width 0.5) (layer "F.Cu") (net 2))
-  (segment (start 111.75 97.145) (end 111.76 97.155) (width 0.5) (layer "F.Cu") (net 2))
-  (segment (start 109.855 91.44) (end 111.76 93.345) (width 0.5) (layer "F.Cu") (net 2))
-  (segment (start 108.345 97.145) (end 108.345 94.605) (width 0.5) (layer "F.Cu") (net 2))
-  (segment (start 111.76 93.345) (end 111.76 97.155) (width 0.5) (layer "F.Cu") (net 2))
-  (segment (start 101.6 98.425) (end 102.86 99.685) (width 0.5) (layer "F.Cu") (net 3))
-  (segment (start 108.345 99.685) (end 108.345 102.225) (width 0.5) (layer "F.Cu") (net 3))
-  (segment (start 102.86 99.685) (end 108.345 99.685) (width 0.5) (layer "F.Cu") (net 3))
-  (segment (start 93.345 98.425) (end 99.645 98.425) (width 0.5) (layer "F.Cu") (net 3))
-  (segment (start 99.645 98.425) (end 101.6 98.425) (width 0.5) (layer "F.Cu") (net 3))
+  (segment (start 91.44 101.6) (end 98.21 101.6) (width 0.5) (layer "F.Cu") (net 1))
+  (segment (start 98.21 101.6) (end 103.53 96.28) (width 0.5) (layer "F.Cu") (net 1))
+  (segment (start 111.76 88.9) (end 114.3 91.44) (width 0.5) (layer "F.Cu") (net 2))
+  (segment (start 114.3 91.44) (end 114.3 95.1) (width 0.5) (layer "F.Cu") (net 2))
+  (segment (start 101.36 91.68) (end 103.53 91.68) (width 0.5) (layer "F.Cu") (net 2))
+  (segment (start 114.3 95.1) (end 120.64 101.44) (width 0.5) (layer "F.Cu") (net 2))
+  (segment (start 103.53 91.68) (end 106.31 88.9) (width 0.5) (layer "F.Cu") (net 2))
+  (segment (start 93.98 99.06) (end 101.36 91.68) (width 0.5) (layer "F.Cu") (net 2))
+  (segment (start 106.31 88.9) (end 111.76 88.9) (width 0.5) (layer "F.Cu") (net 2))
+  (segment (start 123.18 101.84) (end 120.64 101.84) (width 0.5) (layer "F.Cu") (net 2))
+  (segment (start 120.64 101.44) (end 120.64 101.84) (width 0.5) (layer "F.Cu") (net 2))
+  (segment (start 91.44 99.06) (end 93.98 99.06) (width 0.5) (layer "F.Cu") (net 2))
+  (segment (start 118.1 101.84) (end 115.56 101.84) (width 0.5) (layer "F.Cu") (net 3))
+  (segment (start 115.56 99.71) (end 115.56 101.84) (width 0.5) (layer "F.Cu") (net 3))
+  (segment (start 103.53 93.98) (end 109.83 93.98) (width 0.5) (layer "F.Cu") (net 3))
+  (segment (start 109.83 93.98) (end 115.56 99.71) (width 0.5) (layer "F.Cu") (net 3))
 )
